File: placa-pps.kicad_pcb (KiCad board)
At the start: 2 copper layers, 61 x 88.9 mm, 10 parts, among them J1 CONN_01X06, J2 CONN_01X02, Q1 Q_NPN_BCE, Q2 Q_NPN_BCE, Q3 Q_NPN_BCE, U1 Huzzah-Feather, U3 KY-032

Commit message: Correcciones
Parts:
- Q1, Q2, Q3: footprint TO_SOT_Packages_THT:TO-92_Inline_Narrow_Oval -> .pretty:TO-92_NPN
- moved Q1 35.2 mm to (101.6, 95.2), turned to 270 degrees
- moved Q2 34.1 mm to (101.6, 104.1), turned to 270 degrees
- moved R1 33.5 mm to (90.2, 96.5)
- moved Q3 32.9 mm to (101.6, 113.0), turned to 270 degrees
- moved R2 32.4 mm to (90.2, 105.4)
- moved J1 31.2 mm to (92.7, 121.9)
- moved R3 31.2 mm to (90.2, 114.3)
- moved J2 31.2 mm to (105.4, 88.9)
- moved U1 31.2 mm to (105.4, 71.1)
- moved U3 29.0 mm to (67.3, 104.1), turned to 0 degrees
Routing:
- net /SEN: track 42.8 -> 64.4 mm
- net GND: track 0.60 -> 16.6 mm
- net Net-(J1-Pad1): track 44.3 -> 50.9 mm
- net Net-(J1-Pad2): track 35.7 -> 40.2 mm
- net Net-(J1-Pad3): track 19.4 -> 23.4 mm
- net Net-(R1-Pad2): track 22.1 -> 18.8 mm
- net +3V3: track 103.6 -> 106.6 mm
- net /SW: track 88.5 -> 91.2 mm
- net Net-(R2-Pad2): track 36.5 -> 34.5 mm
- net Net-(Q3-Pad1): track 10.2 -> 11.4 mm
- net Net-(Q2-Pad1): track 10.2 -> 11.4 mm
- net Net-(Q1-Pad1): track 10.2 -> 11.4 mm
- net Net-(R3-Pad2): track 46.6 -> 45.9 mm
Other:
- board size 61 x 88.9 mm -> 59.7 x 88.9 mm
- net class Default: trace_width 0.5 -> 0.7

Commit message: Idk
Routing:
- net GND: track 16.6 -> 0.00 mm
Changed lines of the file:
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@@
-(kicad_pcb (version 4) (host pcbnew 4.0.2+dfsg1-stable)
+(kicad_pcb (version 4) (host pcbnew 4.0.6)
   (general
-    (links 0)
+    (links 20)
     (no_connects 0)
-    (area 50.945 45.644999 115.645001 134.695001)
+    (area 51.095 45.644999 114.375001 134.695001)
     (thickness 1.6)
     (drawings 5)
-    (tracks 60)
+    (tracks 56)
     (zones 0)
     (modules 10)
@@
     (mod_text_size 1 1)
     (mod_text_width 0.15)
-    (pad_size 6 6)
-    (pad_drill 2.49936)
+    (pad_size 2 2)
+    (pad_drill 0.7)
     (pad_to_mask_clearance 0.2)
     (aux_axis_origin 85.09 88.9)
     (visible_elements 7FFFEFFF)
     (pcbplotparams
-      (layerselection 0x00030_80000001)
+      (layerselection 0x00000_00000001)
       (usegerberextensions false)
       (excludeedgelayer false)
@@
       (drillshape 2)
       (scaleselection 1)
-      (outputdirectory ""))
+      (outputdirectory C:/Users/Ramiro/Desktop/))
   )
   (net 0 "")
@@
     )
   )
-  (module Pin_Headers:Pin_Header_Straight_1x06_Pitch2.54mm (layer F.Cu)
+  (module Pin_Headers:Pin_Header_Straight_1x06_Pitch2.54mm locked (layer F.Cu)
     (at 92.71 121.92 270)
     (descr "Through hole straight pin header, 1x06, 2.54mm pitch, single row")
@@
       (net 34 "Net-(U3-Pad4)"))
   )
-  (gr_text QSY (at 73.66 66.04) (layer F.Cu)
-    (effects (font (size 4 4) (thickness 0.4)) (justify mirror))
+  (gr_text QSY (at 74.93 66.04) (layer F.Cu)
+    (effects (font (size 4 4) (thickness 0.5)) (justify mirror))
   )
   (gr_line (start 54.61 134.62) (end 54.61 45.72) (angle 90) (layer Edge.Cuts) (width 0.15))
@@
   (segment (start 92.71 121.92) (end 105.41 121.92) (width 0.7) (layer F.Cu) (net 1))
   (segment (start 105.41 121.92) (end 110.49 116.84) (width 0.7) (layer F.Cu) (net 1))
+  (segment (start 90.17 120.65) (end 91.44 119.38) (width 0.7) (layer F.Cu) (net 2))
+  (segment (start 90.17 121.92) (end 90.17 120.65) (width 0.7) (layer F.Cu) (net 2))
   (segment (start 107.95 104.14) (end 106.68 102.87) (width 0.7) (layer F.Cu) (net 2))
   (segment (start 106.68 102.87) (end 101.6 102.87) (width 0.7) (layer F.Cu) (net 2))
   (segment (start 107.95 116.84) (end 107.95 104.14) (width 0.7) (layer F.Cu) (net 2))
-  (segment (start 90.17 120.65) (end 90.17 121.92) (width 0.5) (layer F.Cu) (net 2))
-  (segment (start 91.44 119.38) (end 90.17 120.65) (width 0.7) (layer F.Cu) (net 2))
   (segment (start 105.41 119.38) (end 91.44 119.38) (width 0.7) (layer F.Cu) (net 2))
   (segment (start 107.95 116.84) (end 105.41 119.38) (width 0.7) (layer F.Cu) (net 2))
@@
   (segment (start 87.63 113.03) (end 88.9 111.76) (width 0.7) (layer F.Cu) (net 3))
   (segment (start 88.9 111.76) (end 101.6 111.76) (width 0.7) (layer F.Cu) (net 3))
-  (segment (start 85.09 120.65) (end 85.09 121.92) (width 0.7) (layer F.Cu) (net 4))
-  (segment (start 83.82 119.38) (end 85.09 120.65) (width 0.7) (layer F.Cu) (net 4))
-  (segment (start 77.47 119.38) (end 83.82 119.38) (width 0.7) (layer F.Cu) (net 4))
-  (segment (start 72.39 114.3) (end 77.47 119.38) (width 0.7) (layer F.Cu) (net 4))
   (segment (start 82.55 123.19) (end 82.55 121.92) (width 0.7) (layer F.Cu) (net 5))
   (segment (start 81.28 124.46) (end 82.55 123.19) (width 0.7) (layer F.Cu) (net 5))
@@
     (connect_pads (clearance 0.508))
     (min_thickness 0.254)
-    (fill yes (arc_segments 16) (thermal_gap 0.508) (thermal_bridge_width 0.8) (smoothing chamfer) (radius 2))
+    (fill yes (arc_segments 32) (thermal_gap 0.508) (thermal_bridge_width 0.8) (smoothing chamfer) (radius 2))
     (polygon
       (pts
@@
     (polygon
       (pts
-        (xy 66.04 62.23) (xy 66.04 69.85) (xy 82.55 69.85) (xy 82.55 62.23)
+        (xy 66.839492 62.23) (xy 66.839492 69.85) (xy 83.349492 69.85) (xy 83.349492 62.23)
       )
     )
